File: schematics/BSB-Board.sch (EAGLE design)
At the start: 18 parts, among them Q1 BC107, X1 SSW-106-02-S-S, X2 SSW-116-02-S-S, X3 SSW-108-02-S-S

Commit message: New schematics for Arduino/Raspberry board
Parts:
- removed D3: 1N4148, diode:1N4148DO35-7
- removed JP11, JP12: (no value), SparkFun:M02LOCK
- removed LED1: LED->|, led:LEDSQR2X5
- removed OK1, OK2: 4N25M, optocoupler:4N25M
- removed R4: 287, eagle-ltspice:R0207/10
- removed R5: 374, eagle-ltspice:R0207/10
- removed X1: SSW-106-02-S-S, con-samtec:SSW-106-02-S-S
- removed X2: SSW-116-02-S-S, con-samtec:SSW-116-02-S-S
- removed X3: SSW-108-02-S-S, con-samtec:SSW-108-02-S-S
- added ARD_23-53: (no value), SparkFun-Connectors:M16PTH
- added ARD_8-15: (no value), SparkFun-Connectors:M08
- added ARD_GND, ARD_SUP: (no value), SparkFun-Connectors:M02PTH
- added Q11: BC 557A, transistor-neu-to92:-PNP-TO92-CBE
- added Q12: BC 547A, transistor:BC547-NPN-TO92-CBE
- added R11: 4k7, resistor:R-EU_0204_7
- added R12: 47k, resistor:R-EU_0204_7
- added R13, R14: 10k, resistor:R-EU_0204_7
- added RPI_2-12: (no value), SparkFun-Connectors:M06SILK_FEMALE_PTH
- added SJ1_ARD: Close for Arduino, jumper:SJ
- added SJ3_RPI, SJ4_RPI: Close for RPi, jumper:SJ
- added U1, U2: 4N25, optocoupler:4N25M
- CL: value - CL + -> (none)
- D1: value 1N4148 -> LED->|; device diode:1N4148DO35-7 -> led:LEDSQR2X5
- Q1: value BC107 -> BC 547A; device transistor-npn:BC107 -> transistor:BC547-NPN-TO92-CBE
- R1: value 1k5 -> 560k; device eagle-ltspice:R0207/10 -> resistor:R-EU_0204_7
- R2: value 560k -> 1k5; device eagle-ltspice:R0207/10 -> resistor:R-EU_0204_7
- R3: value 2k2 -> 300; device eagle-ltspice:R0207/10 -> resistor:R-EU_0204_7
Connections:
- removed net A14: R4.2, X3-2.1
- removed net A15: R5.2, X3-1.1
- removed net D23: X2-1.1
- removed net D25: X2-2.1
- removed net D27: X2-3.1
- removed net D29: X2-4.1
- removed net D31: X2-5.1
- removed net D33: X2-6.1
- removed net D35: X2-7.1
- removed net D37: X2-8.1
- removed net D39: X2-9.1
- removed net D41: X2-10.1
- removed net D43: X2-11.1
- removed net D45: X2-12.1
- removed net D47: X2-13.1
- removed net D49: X2-14.1
- removed net D51: X2-15.1
- removed net D53: X2-16.1
- removed net N$10: D2.C, D3.C, JP11.1, JP11.2
- removed net N$13: D3.A, OK2.C
- removed net N$14: JP12.1, JP12.2, R3.2
- removed net N$7: CL-2.KL, D1.C, Q1.E
- removed net N$8: OK1.COL, R3.1, R4.1
- new net 5V-ARD: ARD_SUP.2, SJ1_ARD.2
- new net A14-RXD-ARD: ARD_8-15.2, R11.1, R12.2, U1.COL
- new net A15-TXD-ARD: ARD_8-15.1, Q11.C, R3.2
- new net CL+: CL-1.KL, Q1.C, R2.1, U2.COL
- new net CL-: CL-2.KL, D2.C, Q1.E
- new net GND-ARD: ARD_GND.1, ARD_GND.2, Q12.E, SJ3_RPI.2, U1.EMI, U2.C
- new net GPIO14-TXD-PI: R14.1, RPI_2-12.4
- new net GPIO15-RXD-PI: Q12.C, R13.1, RPI_2-12.5
- new net GPIO18-3V3-PI: RPI_2-12.6, SJ4_RPI.1
- new net PIN6-GND-PI: RPI_2-12.3, SJ3_RPI.1
- new net VCC: Q11.E, R11.2, R13.2, SJ1_ARD.1, SJ4_RPI.2
- net N$1: now also R2.2, U1.A; no longer OK1.A, R1.2
- net N$11: now also R3.1, U2.A; no longer OK2.A, R5.1
- net N$2: now also D1.A, U1.C; no longer LED1.A, OK1.C
- net N$3: now also R1.2, U2.BAS; no longer OK2.BAS, R2.2
- net N$4: now also D1.C, D2.A; no longer D1.A, LED1.C
- net N$5: now also R1.1, U2.EMI; no longer OK2.EMI, R2.1
- net N$6: now also Q12.B, R12.1; no longer CL-1.KL, OK2.COL, Q1.C, R1.1
- net N$9: now also Q11.B, R14.2; no longer D2.A, OK1.EMI
Other:
- note removed: "Ryan Owens"
- moved on the sheet: CL-1, CL-2, D2, Q1, R1, R2, R3
